File: hardware/esparducam-v2/esparducam-v2.brd (EAGLE design)
At the start: 50 x 50 mm, 31 parts, among them J1 FTDI_DEVICE, J2 JST_ZH_3PIN, Q2 MOSFET-PCHANNEL, U1 NCP1117, U2 SPI flash

Commit message: Updated value for C6
Parts:
- C6: value (none) -> 0.1uF
Changed lines of the file:
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@@
 <attribute name="VALUE" x="13.843" y="34.29" size="0.4064" layer="27" font="vector" rot="R180"/>
 </element>
-<element name="C6" library="SparkFun-Capacitors" package="0603-CAP" value="" x="31.369" y="6.604" smashed="yes" rot="R90">
+<element name="C6" library="SparkFun-Capacitors" package="0603-CAP" value="0.1uF" x="31.369" y="6.604" smashed="yes" rot="R90">
 <attribute name="VALUE" x="32.512" y="5.588" size="0.4064" layer="27" font="vector" rot="R90"/>
 </element>
